File: USB-UART.sch (KiCad schematic (older format))
At the start: 22 parts, among them CON1 USB-MICRO-B, P1 CONN_01X03, P2 CONN_01X06, P3 CONN_01X01, U1 FT232RL, U2 ADuM5010-DC/DC-150mW-SSOP20-I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, U3 ADuM3211, U4 ADuM5010-DC/DC-150mW-SSOP20-I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, U5 ADuM3211

Commit message: Change to wire
Connections:
- net at U1.1 (TXD): now also U3.3 (VIB); no longer U3.2 (VOA)
- net at U1.5 (RXD): now also U3.2 (VOA); no longer U3.3 (VIB)
Changed lines of the file:
@@
 P 5550 1525
 F 0 "U4" H 5550 1925 60  0000 C CNN
-F 1 "ADuM5010-DC/DC-150mW-SSOP20-Isolator" H 5550 2050 60  0000 C CNN
+F 1 "ADuM5010-DC/DC-150mW-SSOP20-Isolator" H 5900 325 60  0000 C CNN
 F 2 "Housings_SSOP:SSOP-20_5.3x7.2mm_Pitch0.65mm" H 5425 975 60  0001 C CNN
 F 3 "" H 5425 975 60  0000 C CNN
@@
 P 2075 1525
 F 0 "U2" H 2075 1925 60  0000 C CNN
-F 1 "ADuM5010-DC/DC-150mW-SSOP20-Isolator" H 2075 2050 60  0000 C CNN
+F 1 "ADuM5010-DC/DC-150mW-SSOP20-Isolator" H 2100 175 60  0000 C CNN
 F 2 "Housings_SSOP:SSOP-20_5.3x7.2mm_Pitch0.65mm" H 1950 975 60  0001 C CNN
 F 3 "" H 1950 975 60  0000 C CNN
@@
 	4575 5450 4575 5650
 Connection ~ 4975 5450
-Wire Wire Line
-	6575 3750 7525 3750
-Wire Wire Line
-	7525 3850 6575 3850
 Wire Wire Line
 	7100 3950 7525 3950
@@
 Text Notes 9200 4900 0    60   ~ 0
 Reverse connecting target protection.\nNOTICE: Poly Switch operation time is 1.5s.
+Wire Wire Line
+	6575 3850 7325 3850
+Wire Wire Line
+	7325 3850 7325 3750
+Wire Wire Line
+	7325 3750 7525 3750
+Wire Wire Line
+	6575 3750 7175 3750
+Wire Wire Line
+	7175 3750 7175 3900
+Wire Wire Line
+	7175 3900 7475 3900
+Wire Wire Line
+	7475 3900 7475 3850
+Wire Wire Line
+	7475 3850 7525 3850
 $EndSCHEMATC
